Commit message: Update tetra.xacro

File: tetra_description/urdf/tetra.xacro (robot description, xacro)
@@ -70,5 +70,5 @@
   </link>
   <joint name="camera" type="fixed">
-    <origin xyz="0.135 0.0 0.181" rpy="1.5708 3.14159 1.5708"/>
+    <origin xyz="0.1347 0.0 0.1344" rpy="1.5708 3.14159 1.5708"/> <!--"0.135 0.0 0.181" -->
     <parent link="base_link"/>
     <child link="camera" />
@@ -98,5 +98,5 @@
   </link>
   <joint name="camera1_link" type="fixed">
-    <origin xyz="0.1347 0.0 0.1344" rpy="0 0 0" />
+    <origin xyz="0.1347 0.0 0.1344" rpy="0 0 0"/>
     <parent link="base_link"/>
     <child link="camera1_link" />
